Commit message: New URDF model for Aria V1 arm

File: aria_description/urdf/aria_v1.urdf (robot description, URDF)
Before this commit: robot aria_v1_arm, 10 links, 9 joints
Links:
- removed link C2
- removed link C3
- removed link C4
- removed link C5
- removed link C6
- removed link Finger1+2
- removed link Finger3
- removed link Gripper
- removed link base_link
- added link Band_1, mass 0.47699; collision mesh filename=package://aria_description/meshes/aria_v1/Band_1.STL; visual mesh filename=package://aria_description/meshes/aria_v1/Band_1.STL
- added link Band_2, mass 0.013333; collision mesh filename=package://aria_description/meshes/aria_v1/Band_2.STL; visual mesh filename=package://aria_description/meshes/aria_v1/Band_2.STL
- added link Band_3, mass 0.013333; collision mesh filename=package://aria_description/meshes/aria_v1/Band_3.STL; visual mesh filename=package://aria_description/meshes/aria_v1/Band_3.STL
- added link Band_4, mass 0.010223; collision mesh filename=package://aria_description/meshes/aria_v1/Band_4.STL; visual mesh filename=package://aria_description/meshes/aria_v1/Band_4.STL
- added link Band_5, mass 0.010223; collision mesh filename=package://aria_description/meshes/aria_v1/Band_5.STL; visual mesh filename=package://aria_description/meshes/aria_v1/Band_5.STL
- added link Band_6, mass 0.010223; collision mesh filename=package://aria_description/meshes/aria_v1/Band_6.STL; visual mesh filename=package://aria_description/meshes/aria_v1/Band_6.STL
- added link Link_0, mass 0.47699; collision mesh filename=package://aria_description/meshes/aria_v1/Link_0.STL; visual mesh filename=package://aria_description/meshes/aria_v1/Link_0.STL
- added link Link_1, mass 0.17803; collision mesh filename=package://aria_description/meshes/aria_v1/Link_1.STL; visual mesh filename=package://aria_description/meshes/aria_v1/Link_1.STL
- added link Link_2, mass 0.31497; collision mesh filename=package://aria_description/meshes/aria_v1/Link_2.STL; visual mesh filename=package://aria_description/meshes/aria_v1/Link_2.STL
- added link Link_3, mass 0.15899; collision mesh filename=package://aria_description/meshes/aria_v1/Link_3.STL; visual mesh filename=package://aria_description/meshes/aria_v1/Link_3.STL
- added link Link_4, mass 0.25896; collision mesh filename=package://aria_description/meshes/aria_v1/Link_4.STL; visual mesh filename=package://aria_description/meshes/aria_v1/Link_4.STL
- added link Link_5, mass 0.148; collision mesh filename=package://aria_description/meshes/aria_v1/Link_5.STL; visual mesh filename=package://aria_description/meshes/aria_v1/Link_5.STL
- added link Link_6, mass 0.79487; collision mesh filename=package://aria_description/meshes/aria_v1/Link_6.STL; visual mesh filename=package://aria_description/meshes/aria_v1/Link_6.STL
- added link Link_7(Finger), mass 0.027789; collision mesh filename=package://aria_description/meshes/aria_v1/Link_7(Finger).STL; visual mesh filename=package://aria_description/meshes/aria_v1/Link_7(Finger).STL
- added link Link_8(Finders), mass 0.055822; collision mesh filename=package://aria_description/meshes/aria_v1/Link_8(Finders).S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; visual mesh filename=package://aria_description/meshes/aria_v1/Link_8(Finders).S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
Joints:
- removed joint FJoint1
- removed joint FJoint2
- removed joint Joint1
- removed joint Joint2
- removed joint Joint3
- removed joint Joint4
- removed joint Joint5
- removed joint Joint6
- added joint Band_Joint_1: type fixed, parent Link_0, child Band_1, origin xyz=0 0 0 rpy=0 0 0, axis 0 0 0
- added joint Band_Joint_2: type fixed, parent Link_1, child Band_2, origin xyz=0 0 0 rpy=0 0 0, axis 0 0 0
- added joint Band_Joint_3: type fixed, parent Link_2, child Band_3, origin xyz=0 0 0 rpy=0 0 0, axis 0 0 0
- added joint Band_Joint_4: type fixed, parent Link_3, child Band_4, origin xyz=0 0 0 rpy=0 0 0, axis 0 0 0
- added joint Band_Joint_5: type fixed, parent Link_4, child Band_5, origin xyz=0 0 0 rpy=0 0 0, axis 0 0 0
- added joint Band_Joint_6: type fixed, parent Link_5, child Band_6, origin xyz=0 0 0 rpy=0 0 0, axis 0 0 0
- added joint Joint_1: type continuous, parent Link_0, child Link_1, origin xyz=0 0 0.19525 rpy=0 0 0, axis 0 0 1, limit lower=0 upper=0 effort=0 velocity=0.7
- added joint Joint_2: type revolute, parent Link_1, child Link_2, origin xyz=0 -0.00388 0.11075 rpy=0 0 0, axis 0 -1 0, limit lower=-0.85 upper=3.95 effort=0 velocity=0.9
- added joint Joint_3: type revolute, parent Link_2, child Link_3, origin xyz=0.41 0 0 rpy=0 0 0, axis 0 -1 0, limit lower=-3.22 upper=3.06 effort=0 velocity=0.7
- added joint Joint_4: type continuous, parent Link_3, child Link_4, origin xyz=0.10025 0.01688 0 rpy=0 0 0, axis 1 0 0, limit lower=0 upper=0 effort=0 velocity=1.1
- added joint Joint_5: type revolute, parent Link_4, child Link_5, origin xyz=0.21628 0.00071 -0.05025 rpy=0 0 0, axis 0 -1 0, limit lower=-3.32 upper=1.35 effort=0 velocity=1.1
- added joint Joint_6: type continuous, parent Link_5, child Link_6, origin xyz=0.065533 0.0012125 0.0603 rpy=0 0 0, axis 1 0 0, limit lower=0 upper=0 effort=0 velocity=1.1
- added joint Joint_7: type revolute, parent Link_6, child Link_7(Finger), origin xyz=0.10705 0 0.031 rpy=0 0 0, axis 0 -1 0, limit lower=0 upper=1.06 effort=0 velocity=0.8
- added joint Joint_8: type revolute, parent Link_6, child Link_8(Finders), origin xyz=0.10705 0 -0.031 rpy=0 0 0, axis 0 1 0, limit lower=0 upper=1.06 effort=0 velocity=0.8, mimic joint=Joint_7 multiplier=1 offset=0
- joint eef_joint: parent Gripper -> Link_6

File: aria_description/urdf/aria_v1.urdf.xacro (robot description, xacro)
@@ -8,6 +8,6 @@
   <gazebo>
     <plugin name="finger_2_mimic_joint_plugin" filename="libroboticsgroup_gazebo_mimic_joint_plugin.so">
-      <joint>FJoint1</joint>
-      <mimicJoint>FJoint2</mimicJoint>
+      <joint>Joint_7</joint>
+      <mimicJoint>Joint_8</mimicJoint>
     </plugin>
   </gazebo>
@@ -15,5 +15,5 @@
   <joint name="world_joint" type="fixed">
     <parent link="world" />
-    <child link="base_link" />
+    <child link="Link_0" />
     <origin xyz="0 0 0" rpy="0 0 0" />
   </joint>

File: aria_description/urdf/aria_v1_transmission.xacro (robot description, xacro)
@@ -4,5 +4,5 @@
     <transmission name="arm_trans_1">
       <type>transmission_interface/SimpleTransmission</type>
-      <joint name="Joint1">
+      <joint name="Joint_1">
         <hardwareInterface>hardware_interface/PositionJointInterface</hardwareInterface>
       </joint>
@@ -13,5 +13,5 @@
     <transmission name="arm_trans_2">
       <type>transmission_interface/SimpleTransmission</type>
-      <joint name="Joint2">
+      <joint name="Joint_2">
         <hardwareInterface>hardware_interface/PositionJointInterface</hardwareInterface>
       </joint>
@@ -22,5 +22,5 @@
     <transmission name="arm_trans_3">
       <type>transmission_interface/SimpleTransmission</type>
-      <joint name="Joint3">
+      <joint name="Joint_3">
         <hardwareInterface>hardware_interface/PositionJointInterface</hardwareInterface>
       </joint>
@@ -31,5 +31,5 @@
     <transmission name="arm_trans_4">
       <type>transmission_interface/SimpleTransmission</type>
-      <joint name="Joint4">
+      <joint name="Joint_4">
         <hardwareInterface>hardware_interface/PositionJointInterface</hardwareInterface>
       </joint>
@@ -40,5 +40,5 @@
     <transmission name="arm_trans_5">
       <type>transmission_interface/SimpleTransmission</type>
-      <joint name="Joint5">
+      <joint name="Joint_5">
         <hardwareInterface>hardware_interface/PositionJointInterface</hardwareInterface>
       </joint>
@@ -49,5 +49,5 @@
     <transmission name="arm_trans_6">
       <type>transmission_interface/SimpleTransmission</type>
-      <joint name="Joint6">
+      <joint name="Joint_6">
         <hardwareInterface>hardware_interface/PositionJointInterface</hardwareInterface>
       </joint>
@@ -58,5 +58,5 @@
     <transmission name="finger_trans_1">
       <type>transmission_interface/SimpleTransmission</type>
-      <joint name="FJoint1">
+      <joint name="Joint_7">
         <hardwareInterface>hardware_interface/PositionJointInterface</hardwareInterface>
       </joint>
@@ -67,5 +67,5 @@
     <transmission name="finger_trans_2">
       <type>transmission_interface/SimpleTransmission</type>
-      <joint name="FJoint2">
+      <joint name="Joint_8">
         <hardwareInterface>hardware_interface/PositionJointInterface</hardwareInterface>
       </joint>
