Commit message: support for Aria v2 arm

File: aria_description/urdf/aria_v2.urdf (robot description, URDF)
Before this commit: robot aria_v2_arm, 11 links, 10 joints
Links:
- link arm_link_1: geometry collision mesh filename=package://aria_description/meshes/aria_v2/Link_C2.STL; visual mesh filename=package://aria_description/meshes/aria_v2/Link_C2.STL
- link arm_link_2: geometry collision mesh filename=package://aria_description/meshes/aria_v2/Link_C3.STL; visual mesh filename=package://aria_description/meshes/aria_v2/Link_C3.STL
- link arm_link_3: geometry collision mesh filename=package://aria_description/meshes/aria_v2/Link_C4.STL; visual mesh filename=package://aria_description/meshes/aria_v2/Link_C4.STL
- link arm_link_4: geometry collision mesh filename=package://aria_description/meshes/aria_v2/Link_C5.STL; visual mesh filename=package://aria_description/meshes/aria_v2/Link_C5.STL
- link arm_link_5: geometry collision mesh filename=package://aria_description/meshes/aria_v2/Link_C6.STL; visual mesh filename=package://aria_description/meshes/aria_v2/Link_C6.STL
- link base_link: geometry collision mesh filename=package://aria_description/meshes/aria_v2/base_link.STL; visual mesh filename=package://aria_description/meshes/aria_v2/base_link.STL
- link finger_link_1: geometry collision mesh filename=package://aria_description/meshes/aria_v2/Finger_1.STL; visual mesh filename=package://aria_description/meshes/aria_v2/Finger_1.STL
- link finger_link_2: geometry collision mesh filename=package://aria_description/meshes/aria_v2/Finger_2.STL; visual mesh filename=package://aria_description/meshes/aria_v2/Finger_2.STL
- link finger_link_3: geometry collision mesh filename=package://aria_description/meshes/aria_v2/Finger_3.STL; visual mesh filename=package://aria_description/meshes/aria_v2/Finger_3.STL
- link gripper_link: geometry collision mesh filename=package://aria_description/meshes/aria_v2/Link_Griper.STL; visual mesh filename=package://aria_description/meshes/aria_v2/Link_Griper.STL

Commit message: New URDF model for Aria V2 arm

File: aria_description/urdf/aria_v2.urdf (robot description, URDF)
Before this commit: robot aria_v2_arm, 11 links, 10 joints
Links:
- removed link arm_link_1
- removed link arm_link_2
- removed link arm_link_3
- removed link arm_link_4
- removed link arm_link_5
- removed link base_link
- removed link finger_link_1
- removed link finger_link_2
- removed link finger_link_3
- removed link gripper_link
- added link Band_1, mass 0.53145; collision mesh filename=package://aria_description/meshes/aria_v2/Band_1.STL; visual mesh filename=package://aria_description/meshes/aria_v2/Band_1.STL
- added link Band_2, mass 0.014219; collision mesh filename=package://aria_description/meshes/aria_v2/Band_2.STL; visual mesh filename=package://aria_description/meshes/aria_v2/Band_2.STL
- added link Band_3, mass 0.014219; collision mesh filename=package://aria_description/meshes/aria_v2/Band_3.STL; visual mesh filename=package://aria_description/meshes/aria_v2/Band_3.STL
- added link Band_4, mass 0.012065; collision mesh filename=package://aria_description/meshes/aria_v2/Band_4.STL; visual mesh filename=package://aria_description/meshes/aria_v2/Band_4.STL
- added link Band_5, mass 0.012065; collision mesh filename=package://aria_description/meshes/aria_v2/Band_5.STL; visual mesh filename=package://aria_description/meshes/aria_v2/Band_5.STL
- added link Band_6, mass 0.012065; collision mesh filename=package://aria_description/meshes/aria_v2/Band_6.STL; visual mesh filename=package://aria_description/meshes/aria_v2/Band_6.STL
- added link Link_0, mass 0.53145; collision mesh filename=package://aria_description/meshes/aria_v2/Link_0.STL; visual mesh filename=package://aria_description/meshes/aria_v2/Link_0.STL
- added link Link_1, mass 0.69534; collision mesh filename=package://aria_description/meshes/aria_v2/Link_1.STL; visual mesh filename=package://aria_description/meshes/aria_v2/Link_1.STL
- added link Link_2, mass 1.1208; collision mesh filename=package://aria_description/meshes/aria_v2/Link_2.STL; visual mesh filename=package://aria_description/meshes/aria_v2/Link_2.STL
- added link Link_3, mass 0.59885; collision mesh filename=package://aria_description/meshes/aria_v2/Link_3.STL; visual mesh filename=package://aria_description/meshes/aria_v2/Link_3.STL
- added link Link_4, mass 0.57097; collision mesh filename=package://aria_description/meshes/aria_v2/Link_4.STL; visual mesh filename=package://aria_description/meshes/aria_v2/Link_4.STL
- added link Link_5, mass 0.49438; collision mesh filename=package://aria_description/meshes/aria_v2/Link_5.STL; visual mesh filename=package://aria_description/meshes/aria_v2/Link_5.STL
- added link Link_6, mass 0.59072; collision mesh filename=package://aria_description/meshes/aria_v2/Link_6.STL; visual mesh filename=package://aria_description/meshes/aria_v2/Link_6.STL
- added link Link_7_1, mass 0.0019953; collision mesh filename=package://aria_description/meshes/aria_v2/Link_7_1.STL; visual mesh filename=package://aria_description/meshes/aria_v2/Link_7_1.STL
- added link Link_7_2, mass 0.0065409; collision mesh filename=package://aria_description/meshes/aria_v2/Link_7_2.STL; visual mesh filename=package://aria_description/meshes/aria_v2/Link_7_2.STL
- added link Link_7_3, mass 0.01159; collision mesh filename=package://aria_description/meshes/aria_v2/Link_7_3.STL; visual mesh filename=package://aria_description/meshes/aria_v2/Link_7_3.STL
- added link Link_7_Upper_finger, mass 0.011133; collision mesh filename=package://aria_description/meshes/aria_v2/Link_7_Upper_fing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; visual mesh filename=package://aria_description/meshes/aria_v2/Link_7_Upper_fing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
- added link Link_8_1, mass 0.0039905; collision mesh filename=package://aria_description/meshes/aria_v2/Link_8_1.STL; visual mesh filename=package://aria_description/meshes/aria_v2/Link_8_1.STL
- added link Link_8_2, mass 0.013082; collision mesh filename=package://aria_description/meshes/aria_v2/Link_8_2.STL; visual mesh filename=package://aria_description/meshes/aria_v2/Link_8_2.STL
- added link Link_8_3, mass 0.023181; collision mesh filename=package://aria_description/meshes/aria_v2/Link_8_3.STL; visual mesh filename=package://aria_description/meshes/aria_v2/Link_8_3.STL
- added link Link_8_Lower_fingers, mass 0.022266; collision mesh filename=package://aria_description/meshes/aria_v2/Link_8_Lower_fing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; visual mesh filename=package://aria_description/meshes/aria_v2/Link_8_Lower_fing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
Joints:
- removed joint arm_joint_1
- removed joint arm_joint_2
- removed joint arm_joint_3
- removed joint arm_joint_4
- removed joint arm_joint_5
- removed joint arm_joint_6
- removed joint finger_joint_1
- removed joint finger_joint_2
- removed joint finger_joint_3
- added joint Band_joint_1: type fixed, parent Link_0, child Band_1, origin xyz=0 0 0 rpy=0 0 0, axis 0 0 0
- added joint Band_joint_2: type fixed, parent Link_1, child Band_2, origin xyz=0 0 0 rpy=0 0 0, axis 0 0 0
- added joint Band_joint_3: type fixed, parent Link_2, child Band_3, origin xyz=0 0 0 rpy=0 0 0, axis 0 0 0
- added joint Band_joint_5: type fixed, parent Link_4, child Band_5, origin xyz=0 0 0 rpy=0 0 0, axis 0 0 0
- added joint Band_joint_6: type fixed, parent Link_5, child Band_6, origin xyz=0 0 0 rpy=0 0 0, axis 0 0 0
- added joint Band_joint__4: type fixed, parent Link_3, child Band_4, origin xyz=0 0 0 rpy=0 0 0, axis 0 0 0
- added joint Joint_1: type continuous, parent Link_0, child Link_1, origin xyz=0 0 0.10125 rpy=0 0 0, axis 0 0 1, limit lower=0 upper=0 effort=0 velocity=0.7
- added joint Joint_2: type revolute, parent Link_1, child Link_2, origin xyz=0 0.00025 0.10375 rpy=0 0 0, axis 0 -1 0, limit lower=-0.97 upper=3.615 effort=0 velocity=0.7
- added joint Joint_3: type revolute, parent Link_2, child Link_3, origin xyz=0.41 0 0 rpy=0 0 0, axis 0 -1 0, limit lower=-3.143 upper=1.689 effort=0 velocity=0.7
- added joint Joint_4: type continuous, parent Link_3, child Link_4, origin xyz=0.07925 0.00475 0.03 rpy=0 0 0, axis 1 0 0, limit lower=0 upper=0 effort=0 velocity=1.1
- added joint Joint_5: type revolute, parent Link_4, child Link_5, origin xyz=0.25625 0.01475 0 rpy=0 0 0, axis 0 -1 0, limit lower=-3.14 upper=3.14 effort=0 velocity=1.1
- added joint Joint_6: type continuous, parent Link_5, child Link_6, origin xyz=0.07375 0.03475 0 rpy=0 0 0, axis 1 0 0, limit lower=0 upper=0 effort=0 velocity=1.1
- added joint Joint_7: type revolute, parent Link_6, child Link_7_Upper_finger, origin xyz=0.077886 0 0.030275 rpy=0 0 0, axis 0 -1 0, limit lower=0 upper=1.05 effort=0 velocity=0.4
- added joint Joint_7_1: type fixed, parent Link_7_Upper_finger, child Link_7_1, origin xyz=0 0 0 rpy=0 0 0, axis 0 0 0
- added joint Joint_8: type revolute, parent Link_6, child Link_8_Lower_fingers, origin xyz=0.07921 0 -0.051151 rpy=0 0 0, axis 0 1 0, limit lower=0 upper=1.05 effort=0 velocity=0.4, mimic joint=Joint_7 multiplier=1 offset=0
- added joint Joint_8_1: type fixed, parent Link_8_Lower_fingers, child Link_8_1, origin xyz=0 0 0 rpy=0 0 0, axis 0 0 0
- added joint Joint_8_2: type fixed, parent Link_8_Lower_fingers, child Link_8_2, origin xyz=0 0 0 rpy=0 0 0, axis 0 0 0
- added joint Joint_8_3: type fixed, parent Link_8_Lower_fingers, child Link_8_3, origin xyz=0 0 0 rpy=0 0 0, axis 0 0 0
- added joint Link_7_2: type fixed, parent Link_7_Upper_finger, child Link_7_2, origin xyz=0 0 0 rpy=0 0 0, axis 0 0 0
- added joint Link_7_3: type fixed, parent Link_7_Upper_finger, child Link_7_3, origin xyz=0 0 0 rpy=0 0 0, axis 0 0 0
- joint eef_joint: origin xyz=0.12775 0 0 rpy=3.1415 -1.5708 0 -> xyz=0.1555 0 0 rpy=3.1415 -1.5708 0; parent gripper_link -> Link_6

File: aria_description/urdf/aria_v2.urdf.xacro (robot description, xacro)
@@ -8,12 +8,6 @@
   <gazebo>
     <plugin name="finger_2_mimic_joint_plugin" filename="libroboticsgroup_gazebo_mimic_joint_plugin.so">
-      <joint>finger_joint_1</joint>
-      <mimicJoint>finger_joint_2</mimicJoint>
-    </plugin>
-  </gazebo>
-  <gazebo>
-    <plugin name="finger_3_mimic_joint_plugin" filename="libroboticsgroup_gazebo_mimic_joint_plugin.so">
-      <joint>finger_joint_1</joint>
-      <mimicJoint>finger_joint_3</mimicJoint>
+      <joint>Joint_7</joint>
+      <mimicJoint>Joint_8</mimicJoint>
     </plugin>
   </gazebo>
@@ -21,5 +15,5 @@
   <joint name="world_joint" type="fixed">
     <parent link="world" />
-    <child link="base_link" />
+    <child link="Link_0" />
     <origin xyz="0 0 0" rpy="0 0 0" />
   </joint>

File: aria_description/urdf/aria_v2_transmission.xacro (robot description, xacro)
@@ -4,5 +4,5 @@
     <transmission name="arm_trans_1">
       <type>transmission_interface/SimpleTransmission</type>
-      <joint name="arm_joint_1">
+      <joint name="Joint_1">
         <hardwareInterface>hardware_interface/PositionJointInterface</hardwareInterface>
       </joint>
@@ -13,5 +13,5 @@
     <transmission name="arm_trans_2">
       <type>transmission_interface/SimpleTransmission</type>
-      <joint name="arm_joint_2">
+      <joint name="Joint_2">
         <hardwareInterface>hardware_interface/PositionJointInterface</hardwareInterface>
       </joint>
@@ -22,5 +22,5 @@
     <transmission name="arm_trans_3">
       <type>transmission_interface/SimpleTransmission</type>
-      <joint name="arm_joint_3">
+      <joint name="Joint_3">
         <hardwareInterface>hardware_interface/PositionJointInterface</hardwareInterface>
       </joint>
@@ -31,5 +31,5 @@
     <transmission name="arm_trans_4">
       <type>transmission_interface/SimpleTransmission</type>
-      <joint name="arm_joint_4">
+      <joint name="Joint_4">
         <hardwareInterface>hardware_interface/PositionJointInterface</hardwareInterface>
       </joint>
@@ -40,5 +40,5 @@
     <transmission name="arm_trans_5">
       <type>transmission_interface/SimpleTransmission</type>
-      <joint name="arm_joint_5">
+      <joint name="Joint_5">
         <hardwareInterface>hardware_interface/PositionJointInterface</hardwareInterface>
       </joint>
@@ -49,5 +49,5 @@
     <transmission name="arm_trans_6">
       <type>transmission_interface/SimpleTransmission</type>
-      <joint name="arm_joint_6">
+      <joint name="Joint_6">
         <hardwareInterface>hardware_interface/PositionJointInterface</hardwareInterface>
       </joint>
@@ -58,5 +58,5 @@
     <transmission name="finger_trans_1">
       <type>transmission_interface/SimpleTransmission</type>
-      <joint name="finger_joint_1">
+      <joint name="Joint_7">
         <hardwareInterface>hardware_interface/PositionJointInterface</hardwareInterface>
       </joint>
@@ -67,14 +67,5 @@
     <transmission name="finger_trans_2">
       <type>transmission_interface/SimpleTransmission</type>
-      <joint name="finger_joint_2">
-        <hardwareInterface>hardware_interface/PositionJointInterface</hardwareInterface>
-      </joint>
-      <actuator name="gripper_motor">
-        <mechanicalReduction>1</mechanicalReduction>
-      </actuator>
-    </transmission>
-   <transmission name="finger_trans_3">
-      <type>transmission_interface/SimpleTransmission</type>
-      <joint name="finger_joint_3">
+      <joint name="Joint_8">
         <hardwareInterface>hardware_interface/PositionJointInterface</hardwareInterface>
       </joint>

Commit message: Update aria_v2.urdf, aria_ros_control_udp.cpp, and 3 more files...

File: aria_description/urdf/aria_v2.urdf (robot description, URDF)
Before this commit: robot aria_v2_arm, 22 links, 21 joints
Joints:
- joint Joint_5: type revolute -> continuous
